File: KiCad/VTE346/VTE346.kicad_sch (KiCad schematic)
At the start: 26 parts, among them J1 Power, J3 Program, Q2 IRF540N, SW1 Switch, SW2 Reset, SW3 Mode, U1 AMS1117-3.3, U2 ESP-12F, U3 LM741

Commit message: Updated
Parts:
- removed C1: 100uF, Capacitor_THT:CP_Radial_D5.0mm_P2.50mm, symbol Device:C_Polarized_Small_US
- removed C2: 10uF, Capacitor_THT:CP_Radial_D5.0mm_P2.50mm, symbol Device:C_Polarized_Small_US
- removed D1: 1N4001, Diode_THT:D_A-405_P10.16mm_Horizontal, symbol Device:D_Small
- removed D2: Power, LED_THT:LED_D3.0mm, symbol Device:LED_Small
- removed D3: LED, LED_THT:LED_D3.0mm, symbol Device:LED
- removed D4: 1N4001, Diode_THT:D_DO-41_SOD81_P10.16mm_Horizontal, symbol Diode:1N4001
- removed J3: Program, Connector_PinHeader_2.54mm:PinHeader_1x04_P2.54mm_Vertical, symbol Connector:Conn_01x04_Pin
- removed MK1: Microphone, Buzzer_Beeper:MagneticBuzzer_Kobitone_254-EMB73-RO, symbol Device:Microphone
- removed Q2: IRF540N, Package_TO_SOT_THT:TO-220-3_Vertical, symbol Transistor_FET:IRF540N
- removed R8: 100k, Resistor_THT:R_Axial_DIN0207_L6.3mm_D2.5mm_P10.16mm_Horizontal, symbol Device:R_Small_US
- removed R9: 150, Resistor_THT:R_Axial_DIN0207_L6.3mm_D2.5mm_P10.16mm_Horizontal, symbol Device:R_Small_US
- removed RV1: 10k, Potentiometer_THT:Potentiometer_Runtron_RM-065_Vertical, symbol Device:R_Potentiometer_US
- removed SW1: Switch, TestPoint:TestPoint_2Pads_Pitch2.54mm_Drill0.8mm, symbol Switch:SW_SPST
- removed SW2: Reset, Button_Switch_THT:SW_PUSH_6mm, symbol Switch:SW_SPST
- removed U1: AMS1117-3.3, Package_TO_SOT_SMD:SOT-223-3_TabPin2, symbol Regulator_Linear:AMS1117-3.3
- removed U2: ESP-12F, RF_Module:ESP-12E, symbol RF_Module:ESP-12F
- removed U3: LM741, Package_DIP:DIP-8_W7.62mm_LongPads, symbol Amplifier_Operational:LM741
- added C1: 100nF, Capacitor_THT:C_Disc_D3.0mm_W1.6mm_P2.50mm, symbol Device:C_Small
- added C2, C3: 22pF, Capacitor_THT:C_Disc_D3.0mm_W1.6mm_P2.50mm, symbol Device:C_Small
- added C4, C5: 100uF, Capacitor_THT:CP_Radial_D5.0mm_P2.50mm, symbol Device:C_Polarized_Small_US
- added D1: Red, LED_THT:LED_D3.0mm, symbol Device:LED
- added D2: Green, LED_THT:LED_D3.0mm, symbol Device:LED
- added D3: 1N4001, Diode_THT:D_A-405_P10.16mm_Horizontal, symbol Device:D_Small
- added D4: Power, LED_THT:LED_D3.0mm, symbol Device:LED_Small
- added J2: Program, Connector_PinHeader_2.54mm:PinHeader_1x04_P2.54mm_Vertical, symbol Connector:Conn_01x04_Pin
- added J3: Servo, Connector_PinHeader_2.54mm:PinHeader_1x03_P2.54mm_Vertical, symbol Connector:Conn_01x03_Pin
- added J4: GSM, Connector_PinHeader_2.54mm:PinHeader_1x04_P2.54mm_Vertical, symbol Connector:Conn_01x04_Pin
- added J5: Finger Print, Connector_PinHeader_2.54mm:PinHeader_1x04_P2.54mm_Vertical, symbol Connector:Conn_01x04_Pin
- added Q1: BD138, Package_TO_SOT_THT:TO-126-3_Vertical, symbol Transistor_BJT:BD138
- added SW1: Button, TestPoint:TestPoint_2Pads_Pitch2.54mm_Drill0.8mm, symbol Switch:SW_Push
- added SW2: Reset, Button_Switch_THT:SW_PUSH_6mm, symbol Switch:SW_DPST_x2
- added U1: ATmega328P-P, Package_DIP:DIP-28_W7.62mm_Socket_LongPads, symbol MCU_Microchip_ATmega:ATmega328P-P
- added U2: AMS1117-5.0, Package_TO_SOT_SMD:SOT-223-3_TabPin2, symbol Regulator_Linear:AMS1117-5.0
- added Y1: 16MHz, Crystal:Crystal_HC50_Vertical, symbol Device:Crystal_Small
- BZ1: footprint Connector_PinHeader_2.54mm:PinHeader_1x02_P2.54mm_Vertical -> Buzzer_Beeper:Buzzer_12x9.5RM7.6
- R1: value 1k -> 10k
- R2: value 100k -> 220
- R3: value 10k -> 220
- R4: value 10k -> 100
- R5: value 10k -> 1k
- R6: value 100 -> 3
- SW3: value Mode -> Switch; footprint Button_Switch_THT:SW_PUSH_6mm -> TestPoint:TestPoint_2Pads_Pitch2.54mm_Drill0.8mm
Connections:
- net +12V: now also R5.1, R6.1, C4.1, D3.1 (K), J4.1 (Pin_1), Q1.1 (E); no longer BZ1.1 (+), R1.1
- net GND: now also BZ1.2 (-), C1.2, C2.2, C3.1, C4.2, C5.2, D1.1 (K), D2.1 (K), D4.1 (K), J2.4 (Pin_4), J3.2 (Pin_2), J4.4 (Pin_4), J5.4 (Pin_4), SW1.2, SW2.2 (B), U1.22 (GND), U1.8 (GND), U2.1 (GND); no longer R2.1, R5.2, SW3.2 (B)
- net Rx: now also J2.2 (Pin_2), U1.2 (PD0)
- net Tx: now also J2.3 (Pin_3), U1.3 (PD1)
- net at SW3.1 (A): now also J1.2 (Pin_2); no longer R4.2
- net at R6.2: now also Q1.3 (B), U2.3 (VI)
- net at R2.2: now also D1.2 (A)
- net +5V: now reaches R1.2
- net +5V: now also C5.1, J2.1 (Pin_1), J3.1 (Pin_1), J5.1 (Pin_1), Q1.2 (C), U1.20 (AVCC), U1.7 (VCC), U2.2 (VO)
- net at R3.2: now also D2.2 (A)
- net +3.3V renamed buzzer_pin
- net buzzer_pin: now also U1.26 (PC3); no longer R3.1
- new net: D4.2 (A), R5.2
- new net: R1.1, SW2.1 (A), U1.1 (~{RESET}/PC6)
- new net: D3.2 (A), SW3.2 (B)
- new net: C1.1, U1.21 (AREF)
- new net: C3.2, U1.10 (XTAL2/PB7), Y1.1
- new net: C2.1, U1.9 (XTAL1/PB6), Y1.2
- new net: BZ1.1 (+), R4.2
- new net: SW1.1, U1.5 (PD3)
- new net FP_Rx: J5.2 (Pin_2), U1.14 (PB0)
- new net FP_Tx: J5.3 (Pin_3), U1.13 (PD7)
- new net GSM_Rx: J4.2 (Pin_2), U1.15 (PB1)
- new net GSM_Tx: J4.3 (Pin_3), U1.16 (PB2)
- new net green_pin: R3.1, U1.25 (PC2)
- new net red_pin: R2.1, U1.24 (PC1)
- new net servo: J3.3 (Pin_3), U1.19 (PB5)
- no-connect marks 13 -> 9
