File: KiCad/Ronaldo project/Ronaldo project.kicad_sch (KiCad schematic)
At the start: 24 parts, among them J1 Power, J2 Program, J3 RFID Module, J4 Coin Acceptor, M1 Motor_DC, M2 Motor_DC, SW1 Switch, SW2 Reset, SW3 SW_Push, SW4 SW_Push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

Commit message: New commit to push for the first time
Other:
- moved on the sheet: J2, J4, R5

Commit message: Updates
Parts:
- removed R3, R5, R7: 10k, Resistor_THT:R_Axial_DIN0207_L6.3mm_D2.5mm_P10.16mm_Horizontal, symbol Device:R_Small_US
- removed SW1: Switch, TestPoint:TestPoint_2Pads_Pitch2.54mm_Drill0.8mm, symbol Switch:SW_SPST
- removed SW2: Reset, Button_Switch_THT:SW_PUSH_6mm, symbol Switch:SW_Push_Dual_x2
- removed U3: ESP-12E, RF_Module:ESP-12E, symbol RF_Module:ESP-12E
- added R10, R6, R8, R9: 10k, Resistor_THT:R_Axial_DIN0207_L6.3mm_D2.5mm_P10.16mm_Horizontal, symbol Device:R_Small_US
- added SW5: Reset, Button_Switch_THT:SW_PUSH_6mm, symbol Switch:SW_Push_Dual_x2
- added SW6: Mode, Button_Switch_THT:SW_PUSH_6mm, symbol Switch:SW_Push_Dual_x2
- added U2: ESP-12F, RF_Module:ESP-12E, symbol RF_Module:ESP-12F
- R2: value 10k -> 22k
- R4: value 10k -> 47k
- SW3: value SW_Push -> BTN1
- SW4: value SW_Push -> BTN2
Connections:
- net +3V3: now also SW3.2, SW4.1, R6.2, R9.1, U2.8 (VCC); no longer R2.1, R4.1
- net GND: now also R10.1, R8.2, SW5.1 (C), SW6.2 (D), U2.15 (GND); no longer SW3.1, SW4.1
- net MISO: now also U2.6 (GPIO12)
- net MOSI: now also U2.7 (GPIO13)
- net RST: now also U2.17 (GPIO2)
- net SCK: now also U2.5 (GPIO14)
- net SDA: now also U2.4 (GPIO16)
- net coin: now also R9.2, SW6.1 (C), U2.18 (GPIO0)
- net motor1: now also U2.19 (GPIO4)
- net motor2: now also R8.1, U2.16 (GPIO15)
- net at D1.2 (A): now also J1.1 (Pin_1)
- net at U5.1 (OUT): now also U2.20 (GPIO5)
- net Rx renamed RXD
- net RXD: now also U2.21 (GPIO3/RXD)
- net Tx renamed TXD
- net TXD: now also U2.22 (GPIO1/TXD)
- net button1: no longer names the net of R4.2
- net button1: now also SW4.2; no longer SW3.2
- net button2: no longer names the net of R2.2
- net button2: now also SW3.1; no longer SW4.2
- new net: R10.2, R2.1, R4.1, U2.2 (ADC)
- new net: R6.1, SW5.2 (D), U2.1 (~{RST}), U2.3 (EN)
- no-connect marks 9 -> 12
Other:
- moved on the sheet: C1, C3, D1, D2, J1, J4, M1, M2, R1, R2, R4, SW3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
