File: KiCad/VTE1604 AUTOMATIC TUMBLE DRUM FISH SCALING USING ELECTRIC MOTOR/VTE1604 AUTOMATIC TUMBLE DRUM FISH SCALING USING ELECTRIC MOTOR.kicad_sch (KiCad schematic)
At the start: 24 parts, among them J1 Power, J2 Program, M1 Motor_DC, SW1 Switch, SW2 Reset, SW3 SW_Push, SW4 SW_Push, SW5 SW_Push, U1 ATmega328P-P, U2 AMS1117-5.0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

Commit message: New commit to push for the first time
Connections:
- no-connect marks 11 -> 15
Changed lines of the file:
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@@
+	)
+	(no_connect
+		(at 121.92 90.17)
 	)
 	(no_connect
@@
 	)
 	(no_connect
+		(at 121.92 95.25)
+	)
+	(no_connect
 		(at 199.39 62.23)
 	)
@@
 	(no_connect
 		(at 121.92 143.51)
+	)
+	(no_connect
+		(at 121.92 100.33)
 	)
 	(no_connect
@@
 		(at 200.66 127)
 	)
+	(no_connect
+		(at 121.92 87.63)
+	)
 	(wire

Commit message: Changes
Changed lines of the file:
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@@
 	(wire
 		(pts
-			(xy 198.12 57.15) (xy 198.12 35.56)
+			(xy 195.58 57.15) (xy 195.58 35.56)
 		)
 		(stroke
@@
 	(wire
 		(pts
-			(xy 198.12 35.56) (xy 209.55 35.56)
+			(xy 195.58 35.56) (xy 209.55 35.56)
 		)
 		(stroke
@@
 	(wire
 		(pts
-			(xy 199.39 57.15) (xy 198.12 57.15)
-		)
-		(stroke
+			(xy 199.39 57.15) (xy 195.58 57.15)
+		)
+		(stroke
