File: KiCad/VTE1808/VTE1808.kicad_sch (KiCad schematic)
At the start: 6 parts, among them U1 OP275

Commit message: New commit to push for the first time
Parts:
- removed 1k: R_Small_US, symbol Device:R_Small_US
- removed R, R3: 500, symbol Device:R_Small_US
- removed R3: 5k, symbol Device:R_Small_US
- removed U1: OP275, symbol Amplifier_Operational:OP275
- added BT1: Battery_Cell, Battery:BatteryHolder_Keystone_1058_1x2032, symbol Device:Battery_Cell
- added BZ1: Buzzer, Buzzer_Beeper:Buzzer_12x9.5RM7.6, symbol Device:Buzzer
- added C1, C3: 100uF, Capacitor_THT:CP_Radial_D5.0mm_P2.50mm, symbol Device:C_Polarized_Small_US
- added C2, C6: 100nF, Capacitor_THT:C_Disc_D3.0mm_W1.6mm_P2.50mm, symbol Device:C_Small
- added C4, C5: 22pF, Capacitor_THT:C_Disc_D3.0mm_W1.6mm_P2.50mm, symbol Device:C_Small
- added D1: 1N4001, Diode_THT:D_A-405_P10.16mm_Horizontal, symbol Device:D_Small
- added D2: Power, LED_THT:LED_D3.0mm, symbol Device:LED_Small
- added D3: Ind., LED_THT:LED_D3.0mm, symbol Device:LED_Small
- added J1: Program, Connector_PinHeader_2.54mm:PinHeader_1x04_P2.54mm_Vertical, symbol Connector:Conn_01x04_Pin
- added J2: Display, Connector_PinHeader_2.54mm:PinHeader_1x10_P2.54mm_Vertical, symbol Connector:Conn_01x10_Pin
- added J3: Power, TerminalBlock:TerminalBlock_bornier-2_P5.08mm, symbol Connector:Screw_Terminal_01x02
- added M1: Stepper_Motor, Connector_PinHeader_2.54mm:PinHeader_1x05_P2.54mm_Vertical, symbol Motor:Stepper_Motor_unipolar_5pin
- added R1: 1k, Resistor_THT:R_Axial_DIN0207_L6.3mm_D2.5mm_P10.16mm_Horizontal, symbol Device:R_Small_US
- added R2: 100, Resistor_THT:R_Axial_DIN0207_L6.3mm_D2.5mm_P10.16mm_Horizontal, symbol Device:R_Small_US
- added R3: 10k, Resistor_THT:R_Axial_DIN0207_L6.3mm_D2.5mm_P10.16mm_Horizontal, symbol Device:R_Small_US
- added R4: 220, Resistor_THT:R_Axial_DIN0207_L6.3mm_D2.5mm_P10.16mm_Horizontal, symbol Device:R_Small_US
- added RV1: 1k, Potentiometer_THT:Potentiometer_Runtron_RM-065_Vertical, symbol Device:R_Potentiometer_US
- added SW1: Switch, TestPoint:TestPoint_2Pads_Pitch2.54mm_Drill0.8mm, symbol Switch:SW_SPST
- added SW5, SW6, SW7: SW_Push, TestPoint:TestPoint_2Pads_Pitch2.54mm_Drill0.8mm, symbol Switch:SW_Push
- added SW8: Reset, Button_Switch_THT:SW_PUSH_6mm, symbol Switch:SW_Push
- added U1: AMS1117-5.0, Package_TO_SOT_SMD:SOT-223-3_TabPin2, symbol Regulator_Linear:AMS1117-5.0
- added U2: ATmega328P-P, Package_DIP:DIP-28_W7.62mm_Socket_LongPads, symbol MCU_Microchip_ATmega:ATmega328P-P
- added U3: DS1307+, Package_DIP:DIP-8_W7.62mm, symbol Timer_RTC:DS1307+
- added U5: ULN2003, Package_DIP:DIP-16_W7.62mm_LongPads, symbol Transistor_Array:ULN2003
- added Y1: 16MHz, Crystal:Crystal_HC50_Vertical, symbol Device:Crystal_Small
- added Y2: 32.768kHz, Crystal:Crystal_C26-LF_D2.1mm_L6.5mm_Horizontal, symbol Device:Crystal_Small
- R5: value 1k -> 220; footprint (none) -> Resistor_THT:R_Axial_DIN0207_L6.3mm_D2.5mm_P10.16mm_Horizontal
Connections:
- net GND: now also BT1.2 (-), BZ1.2 (-), C1.2, C2.2, C3.2, C4.2, C5.1, C6.2, D2.1 (K), D3.1 (K), J1.4 (Pin_4), J2.10 (Pin_10), J3.1 (Pin_1), RV1.1, SW5.1, SW6.1, SW7.1, SW8.2, U1.1 (GND), U2.22 (GND), U2.8 (GND), U3.4 (GND), U5.8 (GND)
- net at R5.1: now also J2.7 (Pin_7)
- net +5V: now reaches R5.2
- net +5V: now also C3.1, C6.1, J2.9 (Pin_9), R3.2, RV1.3, U1.2 (VO), U2.20 (AVCC), U2.7 (VCC), U3.8 (VCC)
- new net: D3.2 (A), R4.2
- new net: M1.5, U5.13 (O4)
- new net: M1.4, U5.14 (O3)
- new net: M1.3 (-), U5.15 (O2)
- new net: M1.2, U5.16 (O1)
- new net: C5.2, U2.10 (XTAL2/PB7), Y1.1
- new net: J3.2 (Pin_2), SW1.1 (A)
- new net: D1.2 (A), SW1.2 (B)
- new net: C4.1, U2.9 (XTAL1/PB6), Y1.2
- new net: U3.1 (X1), Y2.1
- new net: U3.2 (X2), Y2.2
- new net: BT1.1 (+), U3.3 (VBAT)
- new net: J2.8 (Pin_8), RV1.2
- new net: D2.2 (A), R1.2
- new net: C2.1, U2.21 (AREF)
- new net: BZ1.1 (+), R2.2
- new net +12V: C1.1, D1.1 (K), M1.1, R1.1, U1.3 (VI), U5.9 (COM)
- new net Backlight: U2.15 (PB1)
- new net Buzzer: R2.1, U2.26 (PC3)
- new net D4: J2.3 (Pin_3), U2.19 (PB5)
- new net D5: J2.4 (Pin_4), U2.18 (PB4)
- new net D6: J2.5 (Pin_5), U2.17 (PB3)
- new net D7: J2.6 (Pin_6), U2.16 (PB2)
- new net E: J2.2 (Pin_2), U2.23 (PC0)
- new net IN1: U2.14 (PB0), U5.1 (I1)
- new net IN2: U2.13 (PD7), U5.2 (I2)
- new net IN3: U2.12 (PD6), U5.3 (I3)
- new net IN4: U2.11 (PD5), U5.4 (I4)
- new net Indicator: R4.1, U2.25 (PC2)
- new net RS: J2.1 (Pin_1), U2.24 (PC1)
- new net Reset: J1.1 (Pin_1), R3.1, SW8.1, U2.1 (~{RESET}/PC6)
- new net Rx: J1.2 (Pin_2), U2.2 (PD0)
- new net SCL: U2.28 (PC5), U3.6 (SCL)
- new net SDA: U2.27 (PC4), U3.5 (SDA)
- new net Tx: J1.3 (Pin_3), U2.3 (PD1)
- new net button1: SW5.2, U2.4 (PD2)
- new net button2: SW6.2, U2.5 (PD3)
- new net button3: SW7.2, U2.6 (PD4)
- no-connect marks 0 -> 7
Other:
- note removed: "Vin"
- note removed: "Vout"

Commit message: latest updated
Changed lines of the file:
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@@
 	(wire
 		(pts
-			(xy 30.48 186.69) (xy 36.83 186.69)
+			(xy 30.48 186.69) (xy 39.37 186.69)
 		)
 		(stroke
@@
 	(wire
 		(pts
-			(xy 30.48 184.15) (xy 38.1 184.15)
+			(xy 30.48 184.15) (xy 39.37 184.15)
 		)
 		(stroke
@@
 	(wire
 		(pts
-			(xy 30.48 181.61) (xy 38.1 181.61)
+			(xy 30.48 181.61) (xy 39.37 181.61)
 		)
 		(stroke
@@
 	)
 	(label "Tx"
-		(at 38.1 184.15 180)
+		(at 39.37 184.15 180)
 		(fields_autoplaced yes)
 		(effects
@@
 	)
 	(label "Rx"
-		(at 38.1 181.61 180)
+		(at 39.37 181.61 180)
 		(fields_autoplaced yes)
 		(effects
@@
 	(symbol
 		(lib_id "power:GND")
-		(at 36.83 186.69 90)
+		(at 39.37 186.69 90)
 		(unit 1)
 		(exclude_from_sim no)
@@
 		(fields_autoplaced yes)
 		(property "Reference" "#PWR03"
-			(at 43.18 186.69 0)
+			(at 45.72 186.69 0)
 			(effects
 				(font
@@
 		)
 		(property "Value" "GND"
-			(at 40.64 186.6899 90)
+			(at 43.18 186.6899 90)
 			(effects
 				(font
@@
 		)
 		(property "Footprint" ""
-			(at 36.83 186.69 0)
+			(at 39.37 186.69 0)
 			(effects
 				(font
@@
 		)
 		(property "Datasheet" ""
-			(at 36.83 186.69 0)
+			(at 39.37 186.69 0)
 			(effects
 				(font
@@
 		)
 		(property "Description" "Power symbol creates a global label with name \"GND\" , ground"
-			(at 36.83 186.69 0)
+			(at 39.37 186.69 0)
 			(effects
 				(font
