File: KiCad/VTE4646: HYBRID RENEWABLE ENERGY MANAGEMENT SYSTEM/VTE4646: HYBRID RENEWABLE ENERGY MANAGEMENT SYSTEM.kicad_sch (KiCad schematic)
At the start: 68 parts, among them J1 Battery 2, J2 Battery 1, J3 Sources, J4 OUTPUT, J5 Programmer, K1 Relay, K2 Relay, Q1 BC547, Q2 BC547, Q3 BC547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

Commit message: Updated
Other:
- moved on the sheet: BZ1, D10, D12, D2, D4, D6, D7, J4, R10, R11, R15, R17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

Commit message: updated
Parts:
- D10: value Green -> LED2
- D12: value Blue -> LED1
Changed lines of the file:
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@@
 			)
 		)
-		(property "Value" "Green"
+		(property "Value" "LED2"
 			(at 230.632 108.712 90)
 			(effects
@@
 			)
 		)
-		(property "Value" "Blue"
+		(property "Value" "LED1"
 			(at 241.3 108.712 90)
 			(effects
