File: KiCad/VTE2657/VTE2657.kicad_pcb (KiCad board)
At the start: 2 copper layers, 65 x 50 mm, 25 parts, among them J1 Program, J2 Power, J3 GSM, J4 Sensor, M1 Stepper_Motor, SW1 Switch, SW2 Reset, SW3 SW_Push, U1 ATmega328P-P, U2 AMS1117-5.0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

Commit message: Updates
Parts:
- added R5: VT93xx, OptoDevice:R_LDR_4.9x4.2mm_P2.54mm_Vertical, F.Cu at (160.1, 93.5)
- added RV1: 10k, Potentiometer_THT:Potentiometer_Runtron_RM-065_Vertical, F.Cu at (162.2, 85.0)
- moved D3 5.62 mm to (160.3, 68.8)
- moved BZ1 0.46 mm to (163.9, 77.5)
Connections:
- U1 pad 24: unconnected-(U1-PC1-Pad24) -> /ldr_pin
Routing:
- net /ldr_pin: track 0.00 -> 51.5 mm
- net +5V: track 80.2 -> 98.6 mm
- net Net-(D3-A): track 9.11 -> 3.81 mm
