File: KiCad/VTE2657/VTE2657.kicad_sch (KiCad schematic)
At the start: 25 parts, among them J1 Program, J2 Power, J3 GSM, J4 Sensor, M1 Stepper_Motor, SW1 Switch, SW2 Reset, SW3 SW_Push, U1 ATmega328P-P, U2 AMS1117-5.0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

Commit message: Updates
Parts:
- added R5: VT93xx, OptoDevice:R_LDR_4.9x4.2mm_P2.54mm_Vertical, symbol Sensor_Optical:VT93xx
- added RV1: 10k, Potentiometer_THT:Potentiometer_Runtron_RM-065_Vertical, symbol Device:R_Potentiometer_US
Connections:
- net +5V: now also RV1.1
- net GND: now also R5.2
- net ldr_pin: now reaches U1.24 (PC1)
- net ldr_pin: now also R5.1, RV1.2, RV1.3
- no-connect marks 14 -> 13
