File: KiCad/VTE5469/VTE5469.kicad_sch (KiCad schematic)
At the start: 34 parts, among them J1 Power, J2 JRD-100 (UHF RFID), J3 Program, J4 Display, Q1 BD138, Q3 BC547, SW1 Switch, SW2 Reset, SW3 Mode, U1 AMS1117-3.3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

Commit message: latest updated
Other:
- moved on the sheet: C1, C2, D1, D2, J1, J2, J3, J4, Q1, R1, R2, R8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

Commit message: Updates
Parts:
- removed U4: Vibration, Sensor_Current:Diodes_SIP-3_4.1x1.5mm_P2.65mm, symbol Sensor_Current:A1369xUA-10
- removed U5: XD-58C, Sensor_Current:Diodes_SIP-3_4.1x1.5mm_P2.65mm, symbol Sensor_Current:A1369xUA-10
- added J5: Vibration, Connector_PinHeader_2.54mm:PinHeader_1x03_P2.54mm_Vertical, symbol Connector:Conn_01x03_Pin
- added J6: XD-58C, Connector_PinHeader_2.54mm:PinHeader_1x03_P2.54mm_Vertical, symbol Connector:Conn_01x03_Pin
Connections:
- net +3.3V: now also J5.1 (Pin_1), J6.2 (Pin_2)
- net +7.4V: now also R6.1
- net GND: now also RV1.1, J5.2 (Pin_2), J6.3 (Pin_3); no longer D3.1 (K), RV1.3
- net frame_pin: now also U2.2 (ADC); no longer U2.9 (CS0)
- net hb_pin: now also U2.7 (GPIO13), J6.1 (Pin_1); no longer U2.2 (ADC)
- net rfid_rx: now also U2.6 (GPIO12); no longer U2.7 (GPIO13)
- net rfid_tx: now also U2.5 (GPIO14); no longer U2.6 (GPIO12)
- net temp_pin: now also U2.17 (GPIO2); no longer U2.11 (GPIO9)
- net vibr_pin: now also R4.2, SW3.1 (A), U2.18 (GPIO0), J5.3 (Pin_3); no longer U2.10 (MISO)
- net mq2: now reaches RV1.2, U3.1 (B1), U3.3 (B2)
- net mq2: now also RV1.3, U2.4 (GPIO16); no longer RV1.1, U2.12 (GPIO10)
- net at U2.16 (GPIO15): now also R5.1, R9.1; no longer R6.1
- net at BZ2.2 (-), D5.2 (A), Q3.1 (C): now also D3.1 (K)
- no-connect marks 3 -> 6
Other:
- moved on the sheet: BZ2, D3, D5, Q3, R5, R6, R7, R9, SW3, U6
