File: KiCad/VTE9413/VTE9413.kicad_sch (KiCad schematic)
At the start: 24 parts, among them J1 Power, J2 Programmer, J3 Flowrate, J4 Flowrate, J5 Display, J6 Motorized valve, J7 Turbidity, J8 PH sensor, Q1 BD138, SW1 Switch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

Commit message: Updates
Connections:
- net flowrate1: now also R8.1, U3.16 (GPIO15); no longer U3.11 (GPIO9)
- net flowrate2: now also U3.17 (GPIO2); no longer U3.12 (GPIO10)
- net ph: now also U3.6 (GPIO12); no longer U3.14 (SCLK)
- net turbidity: now also U3.7 (GPIO13); no longer U3.13 (MOSI)
- net valve_pin1: now also U3.4 (GPIO16); no longer U3.6 (GPIO12)
- net valve_pin2: now also U3.5 (GPIO14); no longer U3.7 (GPIO13)
- no-connect marks 11 -> 12
Other:
- moved on the sheet: C1, C3, D1, D2, J1, J2, J3, J4, J5, J7, J8, Q1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
