File: KiCad/VTE5083: HEART RATE AND DOSAGE MONITORING SYSTEM/VTE5083: HEART RATE AND DOSAGE MONITORING SYSTEM.kicad_pcb (KiCad board)
At the start: 2 copper layers, 57.2 x 45.3 mm, 19 parts, among them J1 Power, J2 Programer, J3 Sensor, SW1 Reset, SW2 Mode, U1 ESP-12E, U2 AMS1117-3.3

Commit message: Changes
Parts:
- removed D3: Red, LED_THT:LED_D3.0mm_Clear
- added J4: ECG sensor, Connector_PinHeader_2.54mm:PinHeader_1x05_P2.54mm_Vertical, F.Cu at (165.7, 66.7)
- added R7: 47k, Resistor_THT:R_Axial_DIN0207_L6.3mm_D2.5mm_P10.16mm_Horizontal, F.Cu at (175.0, 61.1)
- added RV1: 20k, Potentiometer_THT:Potentiometer_Runtron_RM-065_Vertical, F.Cu at (179.4, 76.0)
- added TH1: Thermistor, OptoDevice:Osram_SFH225, F.Cu at (174.5, 79.5)
- D4: value Green -> Red
- J3: value Sensor -> Heartrate sensor
- R5: value 100 -> 20k
- moved D4 34.5 mm to (171.1, 87.6), turned to 90 degrees
- moved C2 17.7 mm to (142.5, 86.3)
- moved SW1 16.0 mm to (154.3, 52.7), turned to 0 degrees
- moved R5 13.1 mm to (164.9, 58.1)
- moved R6 13.0 mm to (171.1, 81.3), turned to 90 degrees
- moved R2 13.0 mm to (175.0, 55.0)
- moved D1 1.97 mm to (147.2, 86.2)
- moved C1 1.81 mm to (161.1, 75.2)
- moved R3 1.71 mm to (138.7, 81.2)
- moved U2 1.60 mm to (165.1, 78.3)
Connections:
- R5 pad 1: Net-(U1-GPIO14) -> /ecg_analog
- R5 pad 2: Net-(D3-A) -> GND
- U1 pad 2: unconnected-(U1-ADC-Pad2) -> /ecg_analog
- U1 pad 4: unconnected-(U1-GPIO16-Pad4) -> /LO-
- U1 pad 5: Net-(U1-GPIO14) -> /LO+
- U1 pad 6: unconnected-(U1-GPIO12-Pad6) -> Net-(U1-GPIO12)
Routing:
- net +3.3V: track 158.8 -> 211.1 mm
- net Net-(U1-GPIO12): track 0.00 -> 29.3 mm
- net /ecg_analog: track 0.00 -> 23.8 mm
- net Net-(U1-GPIO13): track 4.78 -> 20.6 mm
- net Net-(SW1A-B): track 43.2 -> 28.5 mm
- net Net-(D4-A): track 17.9 -> 3.97 mm
- net Net-(D2-K): track 15.1 -> 28.9 mm
- net Net-(D3-A): track 12.6 -> 0.00 mm
- net /LO-: track 0.00 -> 9.93 mm
- net /LO+: track 0.00 -> 5.19 mm
- net GND: track 5.44 -> 10.2 mm, vias 2 -> 4
- net Net-(U1-GPIO14): track 4.54 -> 0.00 mm
- net Net-(RV1-Pad3): track 0.00 -> 3.61 mm
- net Net-(D1-A): track 7.17 -> 5.19 mm
- net Net-(U1-GPIO15): track 26.8 -> 25.8 mm
Other:
- board size 57.2 x 45.3 mm -> 66 x 45.7 mm
