File: KiCad/VTE5083: HEART RATE AND DOSAGE MONITORING SYSTEM/VTE5083: HEART RATE AND DOSAGE MONITORING SYSTEM.kicad_sch (KiCad schematic)
At the start: 19 parts, among them J1 Power, J2 Programer, J3 Sensor, SW1 Reset, SW2 Mode, U1 ESP-12E, U2 AMS1117-3.3

Commit message: latest updated
Connections:
- net at R3.1: now also U1.4 (GPIO16); no longer U1.16 (GPIO15)
- no-connect marks 10 -> 9
Other:
- moved on the sheet: R3
Changed lines of the file:
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@@
-	)
-	(no_connect
-		(at 191.77 102.87)
 	)
 	(no_connect
@@
 	(wire
 		(pts
+			(xy 195.58 105.41) (xy 195.58 102.87)
+		)
+		(stroke
+			(width 0)
+			(type default)
+		)
+	)
+	(wire
+		(pts
 			(xy 134.62 77.47) (xy 138.43 77.47)
 		)
@@
 	(wire
 		(pts
-			(xy 203.2 109.22) (xy 203.2 113.03)
+			(xy 195.58 110.49) (xy 195.58 113.03)
 		)
 		(stroke
@@
 	(wire
 		(pts
-			(xy 191.77 100.33) (xy 203.2 100.33)
-		)
-		(stroke
-			(width 0)
-			(type default)
-		)
-	)
-	(wire
-		(pts
 			(xy 99.06 78.74) (xy 99.06 81.28)
 		)
@@
 	(wire
 		(pts
-			(xy 203.2 100.33) (xy 203.2 104.14)
-		)
-		(stroke
-			(width 0)
-			(type default)
-		)
-	)
-	(wire
-		(pts
 			(xy 111.76 148.59) (xy 124.46 148.59)
 		)
@@
 		(pts
 			(xy 120.65 151.13) (xy 120.65 152.4)
+		)
+		(stroke
+			(width 0)
+			(type default)
+		)
+	)
+	(wire
+		(pts
+			(xy 191.77 102.87) (xy 195.58 102.87)
 		)
 		(stroke
@@
 	(symbol
 		(lib_id "Device:R_Small_US")
-		(at 203.2 106.68 0)
+		(at 195.58 107.95 0)
 		(unit 1)
 		(exclude_from_sim no)
@@
 		(dnp no)
 		(property "Reference" "R3"
-			(at 204.724 105.664 0)
+			(at 197.104 106.934 0)
 			(effects
 				(font
@@
 		)
 		(property "Value" "10k"
-			(at 204.724 107.442 0)
+			(at 197.104 108.712 0)
 			(effects
 				(font
@@
 		)
 		(property "Footprint" "Resistor_THT:R_Axial_DIN0207_L6.3mm_D2.5mm_P10.16mm_Horizontal"
-			(at 203.2 106.68 0)
+			(at 195.58 107.95 0)
 			(effects
 				(font
@@
 		)
 		(property "Datasheet" "~"
-			(at 203.2 106.68 0)
+			(at 195.58 107.95 0)
 			(effects
 				(font
@@
 		)
 		(property "Description" "Resistor, small US symbol"
-			(at 203.2 106.68 0)
+			(at 195.58 107.95 0)
 			(effects
 				(font
@@
 	(symbol
 		(lib_id "power:GND")
-		(at 203.2 113.03 0)
+		(at 195.58 113.03 0)
 		(unit 1)
 		(exclude_from_sim no)
@@
 		(fields_autoplaced yes)
 		(property "Reference" "#PWR013"
-			(at 203.2 119.38 0)
+			(at 195.58 119.38 0)
 			(effects
 				(font
@@
 		)
 		(property "Value" "GND"
-			(at 203.2 118.11 0)
+			(at 195.58 118.11 0)
 			(effects
 				(font
@@
 		)
 		(property "Footprint" ""
-			(at 203.2 113.03 0)
+			(at 195.58 113.03 0)
 			(effects
 				(font
@@
 		)
 		(property "Datasheet" ""
-			(at 203.2 113.03 0)
+			(at 195.58 113.03 0)
 			(effects
 				(font
@@
 		)
 		(property "Description" "Power symbol creates a global label with name \"GND\" , ground"
-			(at 203.2 113.03 0)
-			(effects
-				(font
+			(at 195.58 113.03 0)
+			(effects
+				(font

Commit message: Changes
Parts:
- removed D3: Red, LED_THT:LED_D3.0mm_Clear, symbol Device:LED_Small
- added J4: ECG sensor, Connector_PinHeader_2.54mm:PinHeader_1x05_P2.54mm_Vertical, symbol Connector:Conn_01x05_Pin
- added R7: 47k, Resistor_THT:R_Axial_DIN0207_L6.3mm_D2.5mm_P10.16mm_Horizontal, symbol Device:R_Small_US
- added RV1: 20k, Potentiometer_THT:Potentiometer_Runtron_RM-065_Vertical, symbol Device:R_Potentiometer_US
- added TH1: Thermistor, OptoDevice:Osram_SFH225, symbol Device:Thermistor
- D4: value Green -> Red
- J3: value Sensor -> Heartrate sensor
- R5: value 100 -> 20k
Connections:
- net +3.3V: now also J4.2 (Pin_2), R7.1, RV1.1
- net GND: now also R5.2, J4.1 (Pin_1), TH1.2
- net LO+: now reaches U1.5 (GPIO14)
- net LO+: now also J4.5 (Pin_5); no longer R5.1
- net at R3.1: now also U1.16 (GPIO15); no longer U1.4 (GPIO16)
- net ecg_analog: now reaches U1.2 (ADC)
- net ecg_analog: now also R5.1, J4.3 (Pin_3), R7.2
- net at U1.6 (GPIO12): now also RV1.2
- new net: RV1.3, TH1.1
- new net LO-: J4.4 (Pin_4), U1.4 (GPIO16)
- no-connect marks 9 -> 7
Other:
- moved on the sheet: C1, C2, D1, D2, D4, J1, J2, J3, R1, R2, R3, R4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
