File: KiCad/VTE5083: HEART RATE AND DOSAGE MONITORING SYSTEM/VTE5083: DOSAGE MONITORING SYSTEM/VTE5083: DOSAGE MONITORING SYSTEM.kicad_pcb (KiCad board)
At the start: 2 copper layers, 48.3 x 50.8 mm, 18 parts, among them J1 Power, J3 Programer, SW1 Reset, SW2 Mode, SW3 Button, U1 AMS1117-3.3, U2 ESP-12E

Commit message: Changes
Parts:
- added J2: RTC Module, Connector_PinHeader_2.54mm:PinHeader_1x04_P2.54mm_Vertical, F.Cu at (93.4, 75.2)
- moved SW2 0.88 mm to (95.9, 89.9)
- moved R3 0.50 mm to (106.0, 84.6)
Connections:
- U2 pad 19: unconnected-(U2-GPIO4-Pad19) -> /SDA
- U2 pad 20: unconnected-(U2-GPIO5-Pad20) -> /SCL
Routing:
- net Net-(SW2A-A): track 38.1 -> 29.7 mm
- net /SDA: track 0.00 -> 7.85 mm
- net /SCL: track 0.00 -> 7.62 mm
- net +3.3V: track 165.8 -> 168.2 mm
