File: KiCad/VTE5083: HEART RATE AND DOSAGE MONITORING SYSTEM/VTE5083: DOSAGE MONITORING SYSTEM/VTE5083: DOSAGE MONITORING SYSTEM.kicad_sch (KiCad schematic)
At the start: 18 parts, among them J1 Power, J3 Programer, SW1 Reset, SW2 Mode, SW3 Button, U1 AMS1117-3.3, U2 ESP-12E

Commit message: Changes
Parts:
- added J2: RTC Module, Connector_PinHeader_2.54mm:PinHeader_1x04_P2.54mm_Vertical, symbol Connector:Conn_01x04_Pin
Connections:
- net +3.3V: now also J2.2 (Pin_2)
- net GND: now also J2.1 (Pin_1)
- net SDA: now reaches U2.19 (GPIO4)
- net SDA: now also J2.3 (Pin_3)
- net SCL: now reaches U2.20 (GPIO5)
- net SCL: now also J2.4 (Pin_4)
- no-connect marks 11 -> 9
Other:
- moved on the sheet: BZ1, C1, C2, D1, D2, D3, J1, J3, R1, R2, R3, R4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
