File: KiCad/VTE9934/VTE9934.kicad_sch (KiCad schematic)
At the start: 31 parts, among them J1 MIC, J2 Power, U1 TDA2050, U2 LM741, U3 LM7809_TO220

Commit message: Changes
Changed lines of the file:
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@@
 		(on_board yes)
 		(dnp no)
-		(fields_autoplaced yes)
 		(property "Reference" "R10"
-			(at 86.36 100.33 90)
+			(at 86.36 101.854 90)
 			(effects
 				(font
@@
 		)
 		(property "Value" "22k"
-			(at 86.36 102.87 90)
+			(at 86.106 104.394 90)
 			(effects
 				(font
@@
 		(dnp no)
 		(property "Reference" "R9"
-			(at 70.612 109.22 90)
+			(at 71.12 114.3 90)
 			(effects
 				(font
@@
 		)
 		(property "Value" "47k"
-			(at 70.612 114.3 90)
+			(at 71.12 116.332 90)
 			(effects
 				(font
@@
 		(dnp no)
 		(property "Reference" "C10"
-			(at 78.74 103.124 90)
+			(at 79.502 101.092 90)
 			(effects
 				(font
@@
 		)
 		(property "Value" "0.1uF"
-			(at 80.518 110.236 90)
-			(effects
-				(font
+			(at 80.264 103.378 90)
+			(effects
+				(font
